File: grandiceps.sch (KiCad schematic (older format))
At the start: 88 parts, among them J1 MJ-4PP-9, SW1 ESC, SW10 E, SW11 R, SW12 T, SW13 CAPS, SW14 A, SW15 S, SW16 D, SW17 F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

Commit message: Work on rev2
Changed lines of the file:
@@
 	1    0    0    -1
 $EndComp
+$Comp
+L power:GND #PWR0105
+U 1 1 6045DF73
+P 4125 6625
+F 0 "#PWR0105" H 4125 6375 50  0001 C CNN
+F 1 "GND" H 4130 6452 50  0000 C CNN
+F 2 "" H 4125 6625 50  0001 C CNN
+F 3 "" H 4125 6625 50  0001 C CNN
+	1    4125 6625
+	0    1    1    0
+$EndComp
 $EndSCHEMATC
