File: grandiceps-rev2.kicad_sch (KiCad schematic)
At the start: 106 parts, among them J1 MJ-4PP-9, SW1 ESC, SW10 E, SW11 R, SW12 T, SW13 CAPS, SW14 A, SW15 S, SW16 D, SW17 F, SW18 G, SW19 SHIFT, SW2 1, SW20 <, SW21 Z, SW22 X, SW23 C, SW24 V, SW25 CTRL, SW26 SUPER, SW27 ALT, SW28 X, SW29 C, SW3 2, SW30 Rotary_Encoder_Switch, SW4 3, SW5 4, SW6 5, SW7 TAB, SW8 Q, SW9 W, U1 WeActBlackPill, U2 24LC64

Commit message: Add trackpoint , move thumb
Parts:
- added C10, C11, C12, C13, C14, C15, C16, C17, C18: 100nF, Capacitor_SMD:C_0805_2012Metric, symbol Device:C_Small
- added JP10, JP11, JP12, JP13, JP14, JP15: Jumper_NO_Small, Jumper:SolderJumper-2_P1.3mm_Open_Pad1.0x1.5mm, symbol Device:Jumper_NO_Small
- added U3: PIM447, gcp:pimoroni-trackballl-bommod, symbol grasndiceps:PIM447
Connections:
- net +5V: now also C10.1, C11.1, C12.1, C13.1, C14.1, C15.1, C16.1, C17.1, C18.1, JP12.2, JP13.2
- net GND: now also C10.2, C11.2, C12.2, C13.2, C14.2, C15.2, C16.2, C17.2, C18.2, JP10.2, JP11.2
- net SCL: now also U3.3 (SCL)
- net SDA: now also JP14.2, JP15.2
- new net V: JP10.1, JP13.1, U3.5 (GND)
- new net W: JP11.1, JP12.1, U3.1 (3-5v)
- new net X: JP15.1, U3.4 (INT)
- new net Y: JP14.1, U3.2 (SDA)
