File: bottom/bottom.kicad_pcb (KiCad board)
At the start: 2 copper layers, 149.8 x 115.9 mm, 6 parts

Commit message: update bottom pcb
Parts:
- added G***: LOGO, grandiceps:LOGO, F.Cu at (169.9, 89.2)
- added G***: LOGO, grandiceps:LOGO, B.Cu at (172.3, 89.2)
- H11, H2: value MountingHole -> MountingHole_Pad
Connections:
- H11 pad 1: (no net) -> GND
- H2 pad 1: (no net) -> GND
Routing:
- added copper zone on B.Cu, net (none)
- removed copper zone on B.Cu, net GND
Other:
- net class Default removed

Commit message: Work on rev2
Parts:
- H10, H11, H2, H3, H6, H9: footprint MountingHole:MountingHole_3.2mm_M3 -> MountingHole:MountingHole_2.5mm
Changed lines of the file:
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@@
       (xy -16.336367 -38.889196)) (layer "F.SilkS") (width 0.01) (fill solid))
   )
-  (footprint "MountingHole:MountingHole_3.2mm_M3" (layer "B.Cu")
+  (footprint "MountingHole:MountingHole_2.5mm" (layer "B.Cu")
     (at 196.444 78.486 180)
-    (descr "Mounting Hole 3.2mm, no annular, M3")
-    (tags "mounting hole 3.2mm no annular m3")
+    (descr "Mounting Hole 2.5mm, no annular")
+    (tags "mounting hole 2.5mm no annular")
     (property "Sheetfile" "")
     (property "Sheetname" "")
-    (attr exclude_from_pos_files)
-    (fp_text reference "H2" (at 0 4.2) (layer "B.SilkS")
+    (attr exclude_from_pos_files exclude_from_bom)
+    (fp_text reference "H2" (at 0 3.5) (layer "B.SilkS")
       (effects (font (size 1 1) (thickness 0.15)) (justify mirror))
     )
-    (fp_text value "MountingHole_Pad" (at 0 -4.2) (layer "B.Fab")
+    (fp_text value "MountingHole_Pad" (at 0 -3.5) (layer "B.Fab")
       (effects (font (size 1 1) (thickness 0.15)) (justify mirror))
     )
@@
       (effects (font (size 1 1) (thickness 0.15)) (justify mirror))
     )
-    (fp_circle (center 0 0) (end 3.2 0) (layer "Cmts.User") (width 0.15) (fill none))
-    (fp_circle (center 0 0) (end 3.45 0) (layer "B.CrtYd") (width 0.05) (fill none))
-    (pad "1" np_thru_hole circle (at 0 0 180) (locked) (size 3.2 3.2) (drill 3.2) (layers *.Cu *.Mask)
-      (net 1 "GND") (pinfunction "1") (pintype "input"))
+    (fp_circle (center 0 0) (end 2.5 0) (layer "Cmts.User") (width 0.15) (fill none))
+    (fp_circle (center 0 0) (end 2.75 0) (layer "B.CrtYd") (width 0.05) (fill none))
+    (pad "1" np_thru_hole circle (at 0 0 180) (locked) (size 2.5 2.5) (drill 2.5) (layers *.Cu *.Mask)
+      (net 1 "GND") (pinfunction "1"))
   )
-  (footprint "MountingHole:MountingHole_3.2mm_M3" (layer "B.Cu")
+  (footprint "MountingHole:MountingHole_2.5mm" (layer "B.Cu")
     (at 117.831 105.537 180)
-    (descr "Mounting Hole 3.2mm, no annular, M3")
-    (tags "mounting hole 3.2mm no annular m3")
+    (descr "Mounting Hole 2.5mm, no annular")
+    (tags "mounting hole 2.5mm no annular")
     (attr exclude_from_pos_files exclude_from_bom)
-    (fp_text reference "H3" (at 0 4.2) (layer "B.SilkS")
+    (fp_text reference "H3" (at 0 3.5) (layer "B.SilkS")
       (effects (font (size 1 1) (thickness 0.15)) (justify mirror))
     )
-    (fp_text value "MountingHole" (at 0 -4.2) (layer "B.Fab")
+    (fp_text value "MountingHole" (at 0 -3.5) (layer "B.Fab")
       (effects (font (size 1 1) (thickness 0.15)) (justify mirror))
     )
@@
       (effects (font (size 1 1) (thickness 0.15)) (justify mirror))
     )
-    (fp_circle (center 0 0) (end 3.2 0) (layer "Cmts.User") (width 0.15) (fill none))
-    (fp_circle (center 0 0) (end 3.45 0) (layer "B.CrtYd") (width 0.05) (fill none))
-    (pad "1" np_thru_hole circle (at 0 0 180) (locked) (size 3.2 3.2) (drill 3.2) (layers *.Cu *.Mask))
+    (fp_circle (center 0 0) (end 2.5 0) (layer "Cmts.User") (width 0.15) (fill none))
+    (fp_circle (center 0 0) (end 2.75 0) (layer "B.CrtYd") (width 0.05) (fill none))
+    (pad "1" np_thru_hole circle (at 0 0 180) (locked) (size 2.5 2.5) (drill 2.5) (layers *.Cu *.Mask))
   )
-  (footprint "MountingHole:MountingHole_3.2mm_M3" (layer "B.Cu")
+  (footprint "MountingHole:MountingHole_2.5mm" (layer "B.Cu")
     (at 102.083 128.194 180)
-    (descr "Mounting Hole 3.2mm, no annular, M3")
-    (tags "mounting hole 3.2mm no annular m3")
+    (descr "Mounting Hole 2.5mm, no annular")
+    (tags "mounting hole 2.5mm no annular")
     (attr exclude_from_pos_files exclude_from_bom)
-    (fp_text reference "H9" (at 0 4.2) (layer "B.SilkS")
+    (fp_text reference "H9" (at 0 3.5) (layer "B.SilkS")
       (effects (font (size 1 1) (thickness 0.15)) (justify mirror))
     )
-    (fp_text value "MountingHole" (at 0 -4.2) (layer "B.Fab")
+    (fp_text value "MountingHole" (at 0 -3.5) (layer "B.Fab")
       (effects (font (size 1 1) (thickness 0.15)) (justify mirror))
     )
@@
       (effects (font (size 1 1) (thickness 0.15)) (justify mirror))
     )
-    (fp_circle (center 0 0) (end 3.2 0) (layer "Cmts.User") (width 0.15) (fill none))
-    (fp_circle (center 0 0) (end 3.45 0) (layer "B.CrtYd") (width 0.05) (fill none))
-    (pad "1" np_thru_hole circle (at 0 0 180) (locked) (size 3.2 3.2) (drill 3.2) (layers *.Cu *.Mask))
+    (fp_circle (center 0 0) (end 2.5 0) (layer "Cmts.User") (width 0.15) (fill none))
+    (fp_circle (center 0 0) (end 2.75 0) (layer "B.CrtYd") (width 0.05) (fill none))
+    (pad "1" np_thru_hole circle (at 0 0 180) (locked) (size 2.5 2.5) (drill 2.5) (layers *.Cu *.Mask))
   )
-  (footprint "MountingHole:MountingHole_3.2mm_M3" (layer "B.Cu")
+  (footprint "MountingHole:MountingHole_2.5mm" (layer "B.Cu")
     (at 224.561 133.198 180)
-    (descr "Mounting Hole 3.2mm, no annular, M3")
-    (tags "mounting hole 3.2mm no annular m3")
+    (descr "Mounting Hole 2.5mm, no annular")
+    (tags "mounting hole 2.5mm no annular")
     (attr exclude_from_pos_files exclude_from_bom)
-    (fp_text reference "H10" (at 0 4.2) (layer "B.SilkS")
+    (fp_text reference "H10" (at 0 3.5) (layer "B.SilkS")
       (effects (font (size 1 1) (thickness 0.15)) (justify mirror))
     )
-    (fp_text value "MountingHole" (at 0 -4.2) (layer "B.Fab")
+    (fp_text value "MountingHole" (at 0 -3.5) (layer "B.Fab")
       (effects (font (size 1 1) (thickness 0.15)) (justify mirror))
     )
@@
       (effects (font (size 1 1) (thickness 0.15)) (justify mirror))
     )
-    (fp_circle (center 0 0) (end 3.2 0) (layer "Cmts.User") (width 0.15) (fill none))
-    (fp_circle (center 0 0) (end 3.45 0) (layer "B.CrtYd") (width 0.05) (fill none))
-    (pad "1" np_thru_hole circle (at 0 0 180) (locked) (size 3.2 3.2) (drill 3.2) (layers *.Cu *.Mask))
+    (fp_circle (center 0 0) (end 2.5 0) (layer "Cmts.User") (width 0.15) (fill none))
+    (fp_circle (center 0 0) (end 2.75 0) (layer "B.CrtYd") (width 0.05) (fill none))
+    (pad "1" np_thru_hole circle (at 0 0 180) (locked) (size 2.5 2.5) (drill 2.5) (layers *.Cu *.Mask))
   )
-  (footprint "MountingHole:MountingHole_3.2mm_M3" (layer "B.Cu")
+  (footprint "MountingHole:MountingHole_2.5mm" (layer "B.Cu")
     (at 159.258 79.3496 180)
-    (descr "Mounting Hole 3.2mm, no annular, M3")
-    (tags "mounting hole 3.2mm no annular m3")
+    (descr "Mounting Hole 2.5mm, no annular")
+    (tags "mounting hole 2.5mm no annular")
     (attr exclude_from_pos_files exclude_from_bom)
-    (fp_text reference "H6" (at 0 4.2) (layer "B.SilkS")
+    (fp_text reference "H6" (at 0 3.5) (layer "B.SilkS")
       (effects (font (size 1 1) (thickness 0.15)) (justify mirror))
     )
-    (fp_text value "MountingHole" (at 0 -4.2) (layer "B.Fab")
+    (fp_text value "MountingHole" (at 0 -3.5) (layer "B.Fab")
       (effects (font (size 1 1) (thickness 0.15)) (justify mirror))
     )
@@
       (effects (font (size 1 1) (thickness 0.15)) (justify mirror))
     )
-    (fp_circle (center 0 0) (end 3.2 0) (layer "Cmts.User") (width 0.15) (fill none))
-    (fp_circle (center 0 0) (end 3.45 0) (layer "B.CrtYd") (width 0.05) (fill none))
-    (pad "1" np_thru_hole circle (at 0 0 180) (locked) (size 3.2 3.2) (drill 3.2) (layers *.Cu *.Mask))
+    (fp_circle (center 0 0) (end 2.5 0) (layer "Cmts.User") (width 0.15) (fill none))
+    (fp_circle (center 0 0) (end 2.75 0) (layer "B.CrtYd") (width 0.05) (fill none))
+    (pad "1" np_thru_hole circle (at 0 0 180) (locked) (size 2.5 2.5) (drill 2.5) (layers *.Cu *.Mask))
   )
-  (footprint "MountingHole:MountingHole_3.2mm_M3" (layer "B.Cu")
+  (footprint "MountingHole:MountingHole_2.5mm" (layer "B.Cu")
     (at 93.7766 65.6082 180)
-    (descr "Mounting Hole 3.2mm, no annular, M3")
-    (tags "mounting hole 3.2mm no annular m3")
+    (descr "Mounting Hole 2.5mm, no annular")
+    (tags "mounting hole 2.5mm no annular")
     (property "Sheetfile" "")
     (property "Sheetname" "")
-    (attr exclude_from_pos_files)
-    (fp_text reference "H11" (at 0 4.2) (layer "B.SilkS")
+    (attr exclude_from_pos_files exclude_from_bom)
+    (fp_text reference "H11" (at 0 3.5) (layer "B.SilkS")
       (effects (font (size 1 1) (thickness 0.15)) (justify mirror))
     )
-    (fp_text value "MountingHole_Pad" (at 0 -4.2) (layer "B.Fab")
+    (fp_text value "MountingHole_Pad" (at 0 -3.5) (layer "B.Fab")
       (effects (font (size 1 1) (thickness 0.15)) (justify mirror))
     )
@@
       (effects (font (size 1 1) (thickness 0.15)) (justify mirror))
     )
-    (fp_circle (center 0 0) (end 3.2 0) (layer "Cmts.User") (width 0.15) (fill none))
-    (fp_circle (center 0 0) (end 3.45 0) (layer "B.CrtYd") (width 0.05) (fill none))
-    (pad "1" np_thru_hole circle (at 0 0 180) (locked) (size 3.2 3.2) (drill 3.2) (layers *.Cu *.Mask)
-      (net 1 "GND") (pinfunction "1") (pintype "input"))
+    (fp_circle (center 0 0) (end 2.5 0) (layer "Cmts.User") (width 0.15) (fill none))
+    (fp_circle (center 0 0) (end 2.75 0) (layer "B.CrtYd") (width 0.05) (fill none))
+    (pad "1" np_thru_hole circle (at 0 0 180) (locked) (size 2.5 2.5) (drill 2.5) (layers *.Cu *.Mask)
+      (net 1 "GND") (pinfunction "1"))
   )
   (footprint "grandiceps:LOGO" (layer "B.Cu")
