File: left/left1-rounded.kicad_pcb (KiCad board)
At the start: 2 copper layers, 149.8 x 115.9 mm, 87 parts, among them J1 MJ-4PP-9, SW1 ESC, SW10 E, SW11 R, SW12 T, SW13 CAPS, SW14 A, SW15 S, SW16 D, SW17 F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

Commit message: Work on rev2
Parts:
- added G***: LOGO, grandiceps:Protea-tiny, B.Cu at (196.4, 119.0)
- added G***: LOGO, grandiceps:Protea-tiny, F.Cu at (196.6, 119.0)
