File: left/left1.kicad_pcb (KiCad board)
At the start: 2 copper layers, 149.8 x 115.9 mm, 87 parts, among them J1 MJ-4PP-9, SW1 ESC, SW10 E, SW11 R, SW12 T, SW13 CAPS, SW14 A, SW15 S, SW16 D, SW17 F, SW18 G, SW19 SHIFT, SW2 1, SW20 <, SW21 Z, SW22 X, SW23 C, SW24 V, SW25 CTRL, SW26 SUPER, SW27 ALT, SW28 X, SW29 C, SW3 2, SW30 Rotary_Encoder_Switch, SW4 3, SW5 4, SW6 5, SW7 TAB, SW8 Q, SW9 W, U1 WeActBlackPill

Commit message: Work on rev2
Parts:
- R1: value R_Small -> 10K
Connections:
- U1 pad 30: Net-(U1-Pad30) -> +5V
Routing:
- net +5V: track 411.0 -> 418.4 mm, vias 1 -> 2
Changed lines of the file:
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@@
     (thickness 1.6)
     (drawings 18)
-    (tracks 1450)
+    (tracks 1454)
     (zones 0)
     (modules 87)
-    (nets 78)
+    (nets 77)
   )
   (page A4)
@@
   (net 65 "Net-(J1-PadC)")
   (net 66 "Net-(J1-PadB)")
-  (net 67 "Net-(U1-Pad30)")
-  (net 68 "Net-(U1-Pad29)")
-  (net 69 "Net-(U1-Pad28)")
-  (net 70 "Net-(U1-Pad19)")
-  (net 71 "Net-(U1-Pad18)")
-  (net 72 "Net-(U1-Pad17)")
-  (net 73 "Net-(U1-Pad15)")
-  (net 74 "Net-(U1-Pad14)")
-  (net 75 SCL)
-  (net 76 SDA)
-  (net 77 "Net-(U1-Pad4)")
+  (net 67 "Net-(U1-Pad29)")
+  (net 68 "Net-(U1-Pad28)")
+  (net 69 "Net-(U1-Pad19)")
+  (net 70 "Net-(U1-Pad18)")
+  (net 71 "Net-(U1-Pad17)")
+  (net 72 "Net-(U1-Pad15)")
+  (net 73 "Net-(U1-Pad14)")
+  (net 74 SCL)
+  (net 75 SDA)
+  (net 76 "Net-(U1-Pad4)")
   (net_class Default "This is the default net class."
     (clearance 0.2)
@@
     (add_net "Net-(U1-Pad29)")
     (add_net "Net-(U1-Pad3)")
-    (add_net "Net-(U1-Pad30)")
     (add_net "Net-(U1-Pad32)")
     (add_net "Net-(U1-Pad33)")
@@
       (effects (font (size 1 1) (thickness 0.15)))
     )
-    (fp_text value R_Small (at 2.54 1.92 90) (layer F.Fab)
+    (fp_text value 10K (at 2.54 1.92 90) (layer F.Fab)
       (effects (font (size 1 1) (thickness 0.15)))
     )
@@
       (net 65 "Net-(J1-PadC)"))
     (pad 30 thru_hole circle (at -7.62 20.32) (size 1.524 1.524) (drill 0.762) (layers *.Cu *.Mask)
-      (net 67 "Net-(U1-Pad30)"))
+      (net 2 +5V))
     (pad 29 thru_hole circle (at -7.62 22.86) (size 1.524 1.524) (drill 0.762) (layers *.Cu *.Mask)
-      (net 68 "Net-(U1-Pad29)"))
+      (net 67 "Net-(U1-Pad29)"))
     (pad 28 thru_hole circle (at -7.62 25.4) (size 1.524 1.524) (drill 0.762) (layers *.Cu *.Mask)
-      (net 69 "Net-(U1-Pad28)"))
+      (net 68 "Net-(U1-Pad28)"))
     (pad 27 thru_hole circle (at -7.62 27.94) (size 1.524 1.524) (drill 0.762) (layers *.Cu *.Mask)
-      (net 75 SCL))
+      (net 74 SCL))
     (pad 26 thru_hole circle (at -7.62 30.48) (size 1.524 1.524) (drill 0.762) (layers *.Cu *.Mask)
-      (net 76 SDA))
+      (net 75 SDA))
     (pad 25 thru_hole circle (at -7.62 33.02) (size 1.524 1.524) (drill 0.762) (layers *.Cu *.Mask)
       (net 11 row4))
@@
       (net 62 "Net-(U1-Pad20)"))
     (pad 19 thru_hole circle (at 7.62 40.64) (size 1.524 1.524) (drill 0.762) (layers *.Cu *.Mask)
-      (net 70 "Net-(U1-Pad19)"))
+      (net 69 "Net-(U1-Pad19)"))
     (pad 18 thru_hole circle (at 7.62 38.1) (size 1.524 1.524) (drill 0.762) (layers *.Cu *.Mask)
-      (net 71 "Net-(U1-Pad18)"))
+      (net 70 "Net-(U1-Pad18)"))
     (pad 17 thru_hole circle (at 7.62 35.56) (size 1.524 1.524) (drill 0.762) (layers *.Cu *.Mask)
-      (net 72 "Net-(U1-Pad17)"))
+      (net 71 "Net-(U1-Pad17)"))
     (pad 16 thru_hole circle (at 7.62 33.02) (size 1.524 1.524) (drill 0.762) (layers *.Cu *.Mask))
     (pad 15 thru_hole circle (at 7.62 30.48) (size 1.524 1.524) (drill 0.762) (layers *.Cu *.Mask)
-      (net 73 "Net-(U1-Pad15)"))
+      (net 72 "Net-(U1-Pad15)"))
     (pad 14 thru_hole circle (at 7.62 27.94) (size 1.524 1.524) (drill 0.762) (layers *.Cu *.Mask)
-      (net 74 "Net-(U1-Pad14)"))
+      (net 73 "Net-(U1-Pad14)"))
     (pad 13 thru_hole circle (at 7.62 25.4) (size 1.524 1.524) (drill 0.762) (layers *.Cu *.Mask)
       (net 37 col5))
@@
       (net 63 "Net-(U1-Pad5)"))
     (pad 4 thru_hole circle (at 7.62 2.54) (size 1.524 1.524) (drill 0.762) (layers *.Cu *.Mask)
-      (net 77 "Net-(U1-Pad4)"))
+      (net 76 "Net-(U1-Pad4)"))
     (pad 3 thru_hole circle (at 7.62 0) (size 1.524 1.524) (drill 0.762) (layers *.Cu *.Mask)
       (net 64 "Net-(U1-Pad3)"))
@@
       (net 2 +5V))
     (pad 2 thru_hole circle (at -1.27 0) (size 1.397 1.397) (drill 0.8128) (layers *.Cu F.SilkS B.Mask)
-      (net 75 SCL))
+      (net 74 SCL))
     (pad 1 thru_hole circle (at -3.81 0) (size 1.397 1.397) (drill 0.8128) (layers *.Cu F.SilkS B.Mask)
-      (net 76 SDA))
+      (net 75 SDA))
   )
   (module foostan:MJ-4PP-9 (layer F.Cu)
@@
   (segment (start 157.8355 129.9465) (end 163.322 124.46) (width 0.25) (layer B.Cu) (net 2))
   (segment (start 157.8355 136.246) (end 157.8355 129.9465) (width 0.25) (layer B.Cu) (net 2))
+  (segment (start 172.491 76.6826) (end 176.6824 76.6826) (width 0.25) (layer F.Cu) (net 2))
+  (segment (start 176.6824 76.6826) (end 177.8508 75.5142) (width 0.25) (layer F.Cu) (net 2))
+  (segment (start 177.8508 75.5142) (end 179.4002 75.5142) (width 0.25) (layer F.Cu) (net 2))
+  (via (at 179.4002 75.5142) (size 0.8) (drill 0.4) (layers F.Cu B.Cu) (net 2))
   (segment (start 62.469 54.8726) (end 62.469 54.3726) (width 0.45) (layer B.Cu) (net 3))
   (segment (start 62.173 56.7895) (end 62.469 56.4929) (width 0.45) (layer B.Cu) (net 3))
@@
   (segment (start 193.584 56.5666) (end 192.484 56.5666) (width 0.25) (layer F.Cu) (net 65))
   (segment (start 193.584 53.5666) (end 199.534 53.5666) (width 0.45) (layer F.Cu) (net 66))
-  (segment (start 178.841 105.359) (end 178.841 90.6526) (width 0.25) (layer B.Cu) (net 75))
-  (segment (start 178.841 90.6526) (end 172.491 84.3026) (width 0.25) (layer B.Cu) (net 75))
-  (segment (start 176.301 105.359) (end 176.301 90.6526) (width 0.25) (layer B.Cu) (net 76))
-  (segment (start 176.301 90.6526) (end 172.491 86.8426) (width 0.25) (layer B.Cu) (net 76))
+  (segment (start 178.841 105.359) (end 178.841 90.6526) (width 0.25) (layer B.Cu) (net 74))
+  (segment (start 178.841 90.6526) (end 172.491 84.3026) (width 0.25) (layer B.Cu) (net 74))
+  (segment (start 176.301 105.359) (end 176.301 90.6526) (width 0.25) (layer B.Cu) (net 75))
+  (segment (start 176.301 90.6526) (end 172.491 86.8426) (width 0.25) (layer B.Cu) (net 75))
   (zone (net 1) (net_name GND) (layer F.Cu) (hatch edge 0.508)
     (connect_pads (clearance 0.508))
