File: left/left1.sch (KiCad schematic (older format))
At the start: 88 parts, among them J1 MJ-4PP-9, SW1 ESC, SW10 E, SW11 R, SW12 T, SW13 CAPS, SW14 A, SW15 S, SW16 D, SW17 F, SW18 G, SW19 SHIFT, SW2 1, SW20 <, SW21 Z, SW22 X, SW23 C, SW24 V, SW25 CTRL, SW26 SUPER, SW27 ALT, SW28 X, SW29 C, SW3 2, SW30 Rotary_Encoder_Switch, SW4 3, SW5 4, SW6 5, SW7 TAB, SW8 Q, SW9 W, U1 WeActBlackPill

Commit message: Move folders around
Parts:
- R1: value R_Small -> 10K
Changed lines of the file:
@@
 Text GLabel 4125 7425 0    50   Input ~ 0
 row0
-Text GLabel 5575 6325 2    50   Input ~ 0
+Text GLabel 5575 6725 2    50   Input ~ 0
 row1
 Text GLabel 4125 6325 0    50   Input ~ 0
@@
 Text GLabel 5575 6825 2    50   Input ~ 0
 col1
-Text GLabel 5575 6725 2    50   Input ~ 0
+Text GLabel 5575 6425 2    50   Input ~ 0
 col2
 Text GLabel 5575 6625 2    50   Input ~ 0
@@
 Text GLabel 4125 7625 0    50   Input ~ 0
 ROT1A
-Text GLabel 5575 6425 2    50   Input ~ 0
+Text GLabel 5575 6325 2    50   Input ~ 0
 col5
 NoConn ~ 5575 7025
@@
 P 3350 5000
 F 0 "R1" H 3409 5046 50  0000 L CNN
-F 1 "R_Small" H 3409 4955 50  0000 L CNN
+F 1 "10K" H 3409 4955 50  0000 L CNN
 F 2 "Resistor_THT:R_Axial_DIN0204_L3.6mm_D1.6mm_P5.08mm_Horizontal" H 3350 5000 50  0001 C CNN
 F 3 "~" H 3350 5000 50  0001 C CNN

Commit message: Work on rev2
Changed lines of the file:
@@
 	1    0    0    -1
 $EndComp
+$Comp
+L power:+5V #PWR?
+U 1 1 6045FAAA
+P 4125 6625
+F 0 "#PWR?" H 4125 6475 50  0001 C CNN
+F 1 "+5V" H 4140 6798 50  0000 C CNN
+F 2 "" H 4125 6625 50  0001 C CNN
+F 3 "" H 4125 6625 50  0001 C CNN
+	1    4125 6625
+	0    -1   -1   0
+$EndComp
 $EndSCHEMATC
