File: plate/plate.kicad_pcb (KiCad board)
At the start: 2 copper layers, 149.8 x 115.9 mm, 34 parts, among them SW1 ESC, SW10 E, SW11 R, SW12 T, SW13 CAPS, SW14 A, SW15 S, SW16 D, SW17 F, SW18 G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

Commit message: Work on rev2
Other:
- net class Default removed
