File: rev2/pcb/grandiceps-rev2.kicad_pcb (KiCad board)
At the start: 2 copper layers, 149.9 x 122.6 mm, 122 parts, among them J1 MJ-4PP-9, SW1 ESC, SW10 E, SW11 R, SW12 T, SW13 CAPS, SW14 A, SW15 S, SW16 D, SW17 F, SW18 G, SW19 SHIFT, SW2 1, SW20 <, SW21 Z, SW22 X, SW23 C, SW24 V, SW25 CTRL, SW26 SUPER, SW27 ALT, SW28 X, SW29 C, SW3 2, SW30 Rotary_Encoder_Switch, SW4 3, SW5 4, SW6 5, SW7 TAB, SW8 Q, SW9 W, U1 WeActBlackPill, U2 24LC64, U3 PIM447

Commit message: cleanup
Parts:
- added SW31: Rotary_Encoder_Switch, Grandiceps:RollerEncoder_Panasonic_EVQWGD001, F.Cu at (107.7, 119.2)
Routing:
- net ROT1A: track 99.4 -> 111.2 mm
- net col5: track 129.2 -> 139.2 mm
- net ROT1B: track 93.3 -> 94.9 mm
- net Net-(D30-Pad2): track 17.6 -> 18.5 mm
- net GND: vias 17 -> 18

Commit message: Rev3
Parts:
- moved REF** 27.0 mm to (158.4, 95.2)
Routing:
- net row3: track 145.8 -> 151.1 mm
- net row2: track 179.7 -> 184.3 mm
Other:
- board text added: "Controller in these ------------>"
Changed lines of the file:
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@@
   )
   (footprint "gcp:Tenting_Puck" (layer "F.Cu")
-    (at 177.45 76.15)
+    (at 158.3944 95.2246)
     (attr through_hole)
     (fp_text reference "REF**" (at 7.6835 1.4605) (layer "F.Fab")
@@
   (gr_line (start 238.494865 70.236264) (end 238.494865 60.326464) (layer "Edge.Cuts") (width 0.2))
   (gr_line (start 226.404865 41.620164) (end 234.082865 43.881064) (layer "Edge.Cuts") (width 0.2))
+  (gr_text "Controller\nin these\n------------>" (at 108.9152 56.9214) (layer "B.SilkS")
+    (effects (font (size 1 1) (thickness 0.1)) (justify mirror))
+  )
   (gr_text "RIGHT" (at 92.71 72.39) (layer "F.SilkS")
     (effects (font (size 1 1) (thickness 0.15)))
@@
     (effects (font (size 1 1) (thickness 0.15)))
   )
+  (gr_text "Controller\nin these\n------------>" (at 110.0074 56.769) (layer "F.SilkS")
+    (effects (font (size 1 1) (thickness 0.15)))
+  )
   (via (at 118.45 98.1) (size 0.8) (drill 0.4) (layers "F.Cu" "B.Cu") (net 1))
   (via (at 94.025 83.1) (size 0.8) (drill 0.4) (layers "F.Cu" "B.Cu") (free) (net 1))
@@
   (segment (start 152.883 98.6028) (end 152.3454 98.6028) (width 0.25) (layer "F.Cu") (net 25))
   (segment (start 150.7324 97.5275) (end 151.8077 98.6028) (width 0.25) (layer "F.Cu") (net 25))
+  (segment (start 150.1567 96.9518) (end 142.748 96.9518) (width 0.25) (layer "F.Cu") (net 25))
   (segment (start 102.591 49.7078) (end 116.053 49.7078) (width 0.25) (layer "F.Cu") (net 25))
   (segment (start 209.975 101.325) (end 211.0503 101.325) (width 0.25) (layer "F.Cu") (net 25))
-  (segment (start 152.3454 98.6028) (end 156.5229 94.4253) (width 0.25) (layer "F.Cu") (net 25))
-  (segment (start 132.69 101.016) (end 133.7653 101.016) (width 0.25) (layer "F.Cu") (net 25))
   (segment (start 209.4374 101.325) (end 209.975 101.325) (width 0.25) (layer "F.Cu") (net 25))
   (segment (start 204.0185 96.4438) (end 208.8997 101.325) (width 0.25) (layer "F.Cu") (net 25))
-  (segment (start 137.2538 97.5275) (end 150.7324 97.5275) (width 0.25) (layer "F.Cu") (net 25))
-  (segment (start 156.5229 94.4253) (end 169.8744 94.4253) (width 0.25) (layer "F.Cu") (net 25))
+  (segment (start 171.4874 93.35) (end 170.9497 93.35) (width 0.25) (layer "F.Cu") (net 25))
+  (segment (start 169.875189 94.424511) (end 163.791911 94.424511) (width 0.25) (layer "F.Cu") (net 25))
   (segment (start 180.7704 92.225) (end 172.6124 92.225) (width 0.25) (layer "F.Cu") (net 25))
   (segment (start 211.0503 101.325) (end 212.4346 99.9407) (width 0.25) (layer "F.Cu") (net 25))
   (segment (start 212.4346 99.9407) (end 226.6784 99.9407) (width 0.25) (layer "F.Cu") (net 25))
   (segment (start 190.983 96.4438) (end 184.9892 96.4438) (width 0.25) (layer "F.Cu") (net 25))
-  (segment (start 133.7653 101.016) (end 137.2538 97.5275) (width 0.25) (layer "F.Cu") (net 25))
-  (segment (start 171.4874 93.35) (end 170.9497 93.35) (width 0.25) (layer "F.Cu") (net 25))
   (segment (start 190.983 96.4438) (end 204.0185 96.4438) (width 0.25) (layer "F.Cu") (net 25))
   (segment (start 172.6124 92.225) (end 171.4874 93.35) (width 0.25) (layer "F.Cu") (net 25))
   (segment (start 209.4374 101.325) (end 208.8997 101.325) (width 0.25) (layer "F.Cu") (net 25))
+  (segment (start 142.748 96.9518) (end 141.02895 98.67085) (width 0.25) (layer "F.Cu") (net 25))
+  (segment (start 150.7324 96.6382) (end 150.7324 97.5275) (width 0.25) (layer "F.Cu") (net 25))
   (segment (start 226.6784 99.9407) (end 227.7537 101.016) (width 0.25) (layer "F.Cu") (net 25))
   (segment (start 172.025 93.35) (end 171.4874 93.35) (width 0.25) (layer "F.Cu") (net 25))
   (segment (start 184.9892 96.4438) (end 180.7704 92.225) (width 0.25) (layer "F.Cu") (net 25))
   (segment (start 152.3454 98.6028) (end 151.8077 98.6028) (width 0.25) (layer "F.Cu") (net 25))
-  (segment (start 169.8744 94.4253) (end 170.9497 93.35) (width 0.25) (layer "F.Cu") (net 25))
+  (segment (start 160.867489 91.500089) (end 155.870511 91.500089) (width 0.25) (layer "F.Cu") (net 25))
+  (segment (start 141.02895 98.67085) (end 135.03515 98.67085) (width 0.25) (layer "F.Cu") (net 25))
+  (segment (start 135.03515 98.67085) (end 132.69 101.016) (width 0.25) (layer "F.Cu") (net 25))
+  (segment (start 150.7324 97.5275) (end 150.1567 96.9518) (width 0.25) (layer "F.Cu") (net 25))
+  (segment (start 155.870511 91.500089) (end 150.7324 96.6382) (width 0.25) (layer "F.Cu") (net 25))
+  (segment (start 170.9497 93.35) (end 169.875189 94.424511) (width 0.25) (layer "F.Cu") (net 25))
+  (segment (start 163.791911 94.424511) (end 160.867489 91.500089) (width 0.25) (layer "F.Cu") (net 25))
   (segment (start 118.1074 50.9778) (end 117.323 50.9778) (width 0.25) (layer "B.Cu") (net 25))
   (segment (start 121.1775 91.2654) (end 121.1775 54.0479) (width 0.25) (layer "B.Cu") (net 25))
@@
   (segment (start 150.0663 39.2038) (end 202.9628 39.2038) (width 0.25) (layer "B.Cu") (net 29))
   (segment (start 219.3656 46.8129) (end 218.2903 46.8129) (width 0.25) (layer "B.Cu") (net 29))
-  (segment (start 165.7843 97.5048) (end 167.5261 95.763) (width 0.25) (layer "F.Cu") (net 31))
   (segment (start 120.0054 90.9757) (end 118.1075 89.0778) (width 0.25) (layer "F.Cu") (net 31))
   (segment (start 151.513 99.9) (end 152.756 101.143) (width 0.25) (layer "F.Cu") (net 31))
@@
   (segment (start 172.025 95.763) (end 173.1003 95.763) (width 0.25) (layer "F.Cu") (net 31))
   (segment (start 132.69 103.429) (end 136.219 99.9) (width 0.25) (layer "F.Cu") (net 31))
+  (segment (start 166.1849 97.1042) (end 163.1188 97.1042) (width 0.25) (layer "F.Cu") (net 31))
   (segment (start 136.219 99.9) (end 151.513 99.9) (width 0.25) (layer "F.Cu") (net 31))
   (segment (start 124.6739 102.2) (end 120.0054 97.5315) (width 0.25) (layer "F.Cu") (net 31))
   (segment (start 131.461 102.2) (end 124.6739 102.2) (width 0.25) (layer "F.Cu") (net 31))
-  (segment (start 167.5261 95.763) (end 172.025 95.763) (width 0.25) (layer "F.Cu") (net 31))
+  (segment (start 159.08 101.143) (end 153.8313 101.143) (width 0.25) (layer "F.Cu") (net 31))
   (segment (start 209.6658 103.8652) (end 211.0503 102.4807) (width 0.25) (layer "F.Cu") (net 31))
   (segment (start 209.975 103.8652) (end 209.6658 103.8652) (width 0.25) (layer "F.Cu") (net 31))
   (segment (start 190.983 98.7298) (end 203.7643 98.7298) (width 0.25) (layer "F.Cu") (net 31))
+  (segment (start 172.025 95.763) (end 167.5261 95.763) (width 0.25) (layer "F.Cu") (net 31))
   (segment (start 132.69 103.429) (end 131.461 102.2) (width 0.25) (layer "F.Cu") (net 31))
-  (segment (start 152.756 101.143) (end 153.8313 101.143) (width 0.25) (layer "F.Cu") (net 31))
   (segment (start 175.4373 98.1) (end 180.0714 98.1) (width 0.25) (layer "F.Cu") (net 31))
   (segment (start 203.7643 98.7298) (end 208.8997 103.8652) (width 0.25) (layer "F.Cu") (net 31))
@@
   (segment (start 180.5169 97.6545) (end 188.8324 97.6545) (width 0.25) (layer "F.Cu") (net 31))
   (segment (start 120.0054 97.5315) (end 120.0054 90.9757) (width 0.25) (layer "F.Cu") (net 31))
+  (segment (start 167.5261 95.763) (end 166.1849 97.1042) (width 0.25) (layer "F.Cu") (net 31))
   (segment (start 211.0503 102.4807) (end 226.6784 102.4807) (width 0.25) (layer "F.Cu") (net 31))
   (segment (start 228.829 103.556) (end 227.7537 103.556) (width 0.25) (layer "F.Cu") (net 31))
   (segment (start 188.8324 97.6545) (end 189.9077 98.7298) (width 0.25) (layer "F.Cu") (net 31))
   (segment (start 102.591 87.8078) (end 116.053 87.8078) (width 0.25) (layer "F.Cu") (net 31))
+  (segment (start 159.08 101.143) (end 152.756 101.143) (width 0.25) (layer "F.Cu") (net 31))
   (segment (start 189.9077 98.7298) (end 190.983 98.7298) (width 0.25) (layer "F.Cu") (net 31))
-  (segment (start 153.8313 101.143) (end 157.4695 97.5048) (width 0.25) (layer "F.Cu") (net 31))
-  (segment (start 157.4695 97.5048) (end 165.7843 97.5048) (width 0.25) (layer "F.Cu") (net 31))
   (segment (start 180.0714 98.1) (end 180.5169 97.6545) (width 0.25) (layer "F.Cu") (net 31))
   (segment (start 226.6784 102.4807) (end 227.7537 103.556) (width 0.25) (layer "F.Cu") (net 31))
   (segment (start 209.4374 103.8652) (end 209.6658 103.8652) (width 0.25) (layer "F.Cu") (net 31))
+  (segment (start 163.1188 97.1042) (end 159.08 101.143) (width 0.25) (layer "F.Cu") (net 31))
   (segment (start 209.4374 103.8652) (end 208.8997 103.8652) (width 0.25) (layer "F.Cu") (net 31))
   (segment (start 117.831 61.3902) (end 117.831 62.4078) (width 0.25) (layer "F.Cu") (net 32))
