File: rev2/pcb/grandiceps-rev2.kicad_sch (KiCad schematic)
At the start: 122 parts, among them J1 MJ-4PP-9, SW1 ESC, SW10 E, SW11 R, SW12 T, SW13 CAPS, SW14 A, SW15 S, SW16 D, SW17 F, SW18 G, SW19 SHIFT, SW2 1, SW20 <, SW21 Z, SW22 X, SW23 C, SW24 V, SW25 CTRL, SW26 SUPER, SW27 ALT, SW28 X, SW29 C, SW3 2, SW30 Rotary_Encoder_Switch, SW4 3, SW5 4, SW6 5, SW7 TAB, SW8 Q, SW9 W, U1 WeActBlackPill, U2 24LC64, U3 PIM447

Commit message: cleanup
Parts:
- added SW31: Rotary_Encoder_Switch, Grandiceps:RollerEncoder_Panasonic_EVQWGD001, symbol Device:Rotary_Encoder_Switch
Connections:
- net GND: now also SW31.C
- net ROT1A: now also SW31.A
- net ROT1B: now also SW31.B
- net col5: now also SW31.S2
- net at D30.2 (A), SW30.S1: now also SW31.S1
Changed lines of the file:
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@@
   (junction (at 151.13 62.865) (diameter 1.016) (color 0 0 0 0))
   (junction (at 151.13 75.565) (diameter 1.016) (color 0 0 0 0))
+  (junction (at 166.37 92.71) (diameter 1.016) (color 0 0 0 0))
   (junction (at 173.99 51.435) (diameter 1.016) (color 0 0 0 0))
   (junction (at 173.99 62.865) (diameter 1.016) (color 0 0 0 0))
   (junction (at 173.99 75.565) (diameter 1.016) (color 0 0 0 0))
+  (junction (at 173.99 86.36) (diameter 1.016) (color 0 0 0 0))
   (junction (at 195.58 122.555) (diameter 1.016) (color 0 0 0 0))
   (junction (at 195.58 137.795) (diameter 1.016) (color 0 0 0 0))
@@
     (stroke (width 0) (type solid) (color 0 0 0 0))
   )
-  (wire (pts (xy 166.37 93.98) (xy 166.37 86.36))
+  (wire (pts (xy 166.37 92.71) (xy 166.37 86.36))
+    (stroke (width 0) (type solid) (color 0 0 0 0))
+  )
+  (wire (pts (xy 166.37 92.71) (xy 182.245 92.71))
+    (stroke (width 0) (type solid) (color 0 0 0 0))
+  )
+  (wire (pts (xy 166.37 93.98) (xy 166.37 92.71))
     (stroke (width 0) (type solid) (color 0 0 0 0))
   )
@@
     (stroke (width 0) (type solid) (color 0 0 0 0))
   )
+  (wire (pts (xy 187.325 86.36) (xy 173.99 86.36))
+    (stroke (width 0) (type solid) (color 0 0 0 0))
+  )
+  (wire (pts (xy 187.325 92.71) (xy 187.325 86.36))
+    (stroke (width 0) (type solid) (color 0 0 0 0))
+  )
   (wire (pts (xy 193.675 196.85) (xy 203.835 196.85))
     (stroke (width 0) (type solid) (color 0 0 0 0))
@@
     )
   )
+  (global_label "ROT1A" (shape input) (at 182.245 107.95 270) (fields_autoplaced)
+    (effects (font (size 1.27 1.27)) (justify right))
+    (property "Intersheet References" "${INTERSHEET_REFS}" (id 0) (at 15.875 -1.27 0)
+      (effects (font (size 1.27 1.27)) hide)
+    )
+  )
+  (global_label "ROT1B" (shape input) (at 187.325 107.95 270) (fields_autoplaced)
+    (effects (font (size 1.27 1.27)) (justify right))
+    (property "Intersheet References" "${INTERSHEET_REFS}" (id 0) (at 15.875 -1.27 0)
+      (effects (font (size 1.27 1.27)) hide)
+    )
+  )
   (global_label "RGB" (shape input) (at 187.96 130.175 180) (fields_autoplaced)
     (effects (font (size 1.27 1.27)) (justify right))
@@
     (pin "1")
   )
+  (symbol (lib_id "power:GND") (at 184.785 107.95 0) (unit 1)
+    (in_bom yes) (on_board yes)
+    (property "Reference" "#PWR0111" (id 0) (at 184.785 114.3 0)
+      (effects (font (size 1.27 1.27)) hide)
+    )
+    (property "Value" "GND" (id 1) (at 184.912 112.3442 0))
+    (property "Footprint" "" (id 2) (at 184.785 107.95 0)
+      (effects (font (size 1.27 1.27)) hide)
+    )
+    (property "Datasheet" "" (id 3) (at 184.785 107.95 0)
+      (effects (font (size 1.27 1.27)) hide)
+    )
+    (pin "1")
+  )
   (symbol (lib_id "power:GND") (at 195.58 137.795 0) (unit 1)
     (in_bom yes) (on_board yes)
@@
     (pin "S2")
   )
+  (symbol (lib_id "Device:Rotary_Encoder_Switch") (at 184.785 100.33 90) (unit 1)
+    (in_bom yes) (on_board yes)
+    (property "Reference" "SW31" (id 0) (at 175.4632 100.33 0))
+    (property "Value" "Rotary_Encoder_Switch" (id 1) (at 177.7746 100.33 0))
+    (property "Footprint" "Grandiceps:RollerEncoder_Panasonic_EVQWGD001" (id 2) (at 180.721 104.14 0)
+      (effects (font (size 1.27 1.27)) hide)
+    )
+    (property "Datasheet" "~" (id 3) (at 178.181 100.33 0)
+      (effects (font (size 1.27 1.27)) hide)
+    )
+    (pin "A")
+    (pin "B")
+    (pin "C")
+    (pin "S1")
+    (pin "S2")
+  )
   (symbol (lib_id "LED:WS2812B") (at 195.58 130.175 0) (unit 1)
     (in_bom yes) (on_board yes)
@@
       (reference "#PWR0110") (unit 1) (value "GND") (footprint "")
     )
+    (path "/795b72b5-7451-45f4-bbbd-dc7676d97108"
+      (reference "#PWR0111") (unit 1) (value "GND") (footprint "")
+    )
     (path "/00000000-0000-0000-0000-00005fc6c7af"
       (reference "C1") (unit 1) (value "100nF") (footprint "Capacitor_SMD:C_0805_2012Metric")
@@
       (reference "SW30") (unit 1) (value "Rotary_Encoder_Switch") (footprint "Rotary_Encoder:RotaryEncoder_Alps_EC11E-Switch_Vertical_H20mm")
     )
+    (path "/2d1d707d-9d67-4cc0-8220-e83de7663c1e"
+      (reference "SW31") (unit 1) (value "Rotary_Encoder_Switch") (footprint "Grandiceps:RollerEncoder_Panasonic_EVQWGD001")
+    )
     (path "/00000000-0000-0000-0000-00006023b198"

Commit message: Rev3
Parts:
- added SW32: Rotary_Encoder_Switch, Grandiceps:RollerEncoder_Panasonic_EVQWGD001, symbol Device:Rotary_Encoder_Switch
Connections:
- net GND: now also SW32.C
- net ROT1A: now also SW32.A
- net ROT1B: now also SW32.B
- net col5: now also SW32.S2
- net at D30.2 (A), SW30.S1, SW31.S1: now also SW32.S1
