File: rev2/plate/grandiceps-rev2-plate.kicad_pcb (KiCad board)
At the start: 2 copper layers, 149.9 x 122.6 mm, 35 parts, among them SW1 ESC, SW10 E, SW11 R, SW12 T, SW13 CAPS, SW14 A, SW15 S, SW16 D, SW17 F, SW18 G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

Commit message: Rev3
Other:
- outline, holes or cut-outs redrawn
Changed lines of the file:
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@@
-(kicad_pcb (version 20210424) (generator pcbnew)
+(kicad_pcb (version 20210722) (generator pcbnew)
   (general
     (thickness 1.6)
@@
   )
   (gr_arc (start 222.282835 131.100845) (end 224.535523 140.839973) (angle -34.80768632) (layer "Edge.Cuts") (width 0.2))
+  (gr_line (start 120.5738 100.965) (end 114.7826 100.9396) (layer "Edge.Cuts") (width 0.2))
+  (gr_line (start 114.7826 105.41) (end 99.6442 105.41) (layer "Edge.Cuts") (width 0.2))
+  (gr_line (start 120.5992 43.4848) (end 120.5738 100.965) (layer "Edge.Cuts") (width 0.2))
   (gr_line (start 89.8404 146.5752) (end 93.654382 153.534802) (layer "Edge.Cuts") (width 0.2))
   (gr_line (start 88.675193 110.967367) (end 88.6754 123.3342) (layer "Edge.Cuts") (width 0.2))
@@
   (gr_arc (start 204.488 114.9722) (end 229.691781 137.811489) (angle -45.25337) (layer "Edge.Cuts") (width 0.2))
   (gr_line (start 142.165 102.5152) (end 156.165 102.5152) (layer "Edge.Cuts") (width 0.2))
-  (gr_arc (start 177.293 258.4232) (end 226.417039 41.637323) (angle -27.7477) (layer "Edge.Cuts") (width 0.2))
-  (gr_line (start 118.012 100.9672) (end 118.012 45.6922) (layer "Edge.Cuts") (width 0.2))
+  (gr_arc (start 177.278016 258.489222) (end 226.417039 41.637323) (angle -27.53586562) (layer "Edge.Cuts") (width 0.2))
   (gr_line (start 238.507 70.2535) (end 238.507 60.3437) (layer "Edge.Cuts") (width 0.2))
-  (gr_line (start 118.012 45.6922) (end 119.662 45.6755) (layer "Edge.Cuts") (width 0.2))
+  (gr_line (start 98.675193 100.9672) (end 99.6442 100.9396) (layer "Edge.Cuts") (width 0.2))
+  (gr_line (start 114.7826 105.41) (end 114.7826 100.9396) (layer "Edge.Cuts") (width 0.2))
   (gr_line (start 142.165 116.5152) (end 142.165 102.5152) (layer "Edge.Cuts") (width 0.2))
   (gr_line (start 88.6754 123.3342) (end 88.610062 141.734769) (layer "Edge.Cuts") (width 0.2))
@@
   (gr_arc (start 187.258469 351.913398) (end 189.077658 143.52874) (angle -15.5851766) (layer "Edge.Cuts") (width 0.2))
   (gr_line (start 133.023934 150.701842) (end 105.07 158.3732) (layer "Edge.Cuts") (width 0.2))
-  (gr_line (start 119.662 45.6755) (end 119.837135 43.695206) (layer "Edge.Cuts") (width 0.2))
   (gr_line (start 156.165 102.5152) (end 156.165 116.5152) (layer "Edge.Cuts") (width 0.2))
   (gr_line (start 114.737 126.5172) (end 99.687 126.5172) (layer "Edge.Cuts") (width 0.2))
-  (gr_line (start 98.675193 100.9672) (end 118.012 100.9672) (layer "Edge.Cuts") (width 0.2))
   (gr_line (start 99.687 126.5172) (end 99.687 108.4172) (layer "Edge.Cuts") (width 0.2))
   (gr_line (start 156.165 116.5152) (end 142.165 116.5152) (layer "Edge.Cuts") (width 0.2))
   (gr_line (start 99.687 108.4172) (end 114.737 108.4172) (layer "Edge.Cuts") (width 0.2))
   (gr_line (start 238.504 50.974) (end 238.507 52.9223) (layer "Edge.Cuts") (width 0.2))
+  (gr_line (start 99.6442 105.41) (end 99.6442 100.9396) (layer "Edge.Cuts") (width 0.2))
   (zone (net 1) (net_name "GND") (layer "F.Cu") (hatch edge 0.508)
     (connect_pads (clearance 0.508))
